File: hardware/kicad/radxa_zero3w_robot_hat.kicad_sch (KiCad schematic)
At the start: 6 parts

Commit message: [verified] feat(hardware): restore full Robot HAT connector parity
Other:
- note added: "Radxa ZERO 3W host allocation: - I2C3 M0 pins 3/5: IMU + Audio + Qwiic J5 - UART2 M0 pins 8/10: Dynamixel half-duplex - I2S3 M0 pins 12/35/38/40: Audio - I2C4/USB alternate pins 27/28: upstream HAT-ID path, U4 DNP - Qwiic J6/J7/J8: independent i2c-gpio aliases 10/11/12 See 09_STRICT_PORT_CHANGE_MATRIX.md and the Radxa device-tree notes."
- note removed: "Radxa ZERO 3W host allocation: - I2C3 M0 pins 3/5: IMU + Audio + Qwiic J5 - UART2 M0 pins 8/10: Dynamixel half-duplex - I2S3 M0 pins 12/35/38/40: Audio - I2C4/USB alternate pins 27/28: upstream HAT-ID path, U4 DNP - Pi-specific auxiliary Qwiic connectors J6/J7/J8: DNP See 09_STRICT_PORT_CHANGE_MATRIX.md and the Radxa device-tree notes."
Changed lines of the file:
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@@
 		)
 	)
-	(text "Radxa ZERO 3W host allocation:\n- I2C3 M0 pins 3/5: IMU + Audio + Qwiic J5\n- UART2 M0 pins 8/10: Dynamixel half-duplex\n- I2S3 M0 pins 12/35/38/40: Audio\n- I2C4/USB alternate pins 27/28: upstream HAT-ID path, U4 DNP\n- Pi-specific auxiliary Qwiic connectors J6/J7/J8: DNP\nSee 09_STRICT_PORT_CHANGE_MATRIX.md and the Radxa device-tree notes."
+	(text "Radxa ZERO 3W host allocation:\n- I2C3 M0 pins 3/5: IMU + Audio + Qwiic J5\n- UART2 M0 pins 8/10: Dynamixel half-duplex\n- I2S3 M0 pins 12/35/38/40: Audio\n- I2C4/USB alternate pins 27/28: upstream HAT-ID path, U4 DNP\n- Qwiic J6/J7/J8: independent i2c-gpio aliases 10/11/12\nSee 09_STRICT_PORT_CHANGE_MATRIX.md and the Radxa device-tree notes."
 		(exclude_from_sim no)
 		(at 181.102 57.912 0)

Commit message: [verified] feat(hardware): remove upstream brand logos
Parts:
- removed H2: Logo HF 2025, Library_Pollen:Logo_HF_2025, symbol Library_Pollen:Logo HF 2025
- removed H3: DNP Logo Pollen 2021, Library_Pollen:Logo_Pollen_2021_sq, symbol Library_Pollen:Logo Pollen 2021
