File: hardware/kicad/radxa_zero3w_robot_hat.kicad_pcb (KiCad board)
At the start: 4 copper layers, 65 x 30.9 mm, 128 parts, among them J1 Wago-2, J11 Dynamixel-4, J13 Dynamixel-3, J14 Dynamixel-3, J2 Wago-2, J3 Dynamixel-4, J4 Radxa ZERO 3W 2x20 HAT Header, J5 JST SH, J6 JST SH, J7 JST SH, J8 JST SH, J9 Wago-2, Q1 MMBT3906, Q2 SI2312CDS-T1-GE3, U1 PAM8406D, U10 LM5050-1, U11 BMI088, U2 TLV320AIC3104IRHBR, U3 XC6206P182MR, U4 DNP-CAT24C32HU4, U5 74LVC1G08, U6 SN74LVC1G125DBV, U7 SN74LVC1G126DBVR, U8 SIT3088E, U9 AP63205, Y1 12 MHz

Commit message: [verified] feat(hardware): restore full Robot HAT connector parity
Parts:
- R18, R19: value DNP-0R -> 0R
- R20, R21, R34, R35, R38, R39: value DNP-10k -> 10k
Changed lines of the file:
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@@
 		(sheetname "/Schematic/Sensors/")
 		(sheetfile "sensors.kicad_sch")
-		(attr smd dnp)
+		(attr smd)
 		(fp_line
 			(start 3.11 1.11)
@@
 			)
 		)
-		(property "Value" "DNP-0R"
+		(property "Value" "0R"
 			(at 0 1.17 0)
 			(layer "F.Fab")
@@
 		(sheetname "/Schematic/Sensors/")
 		(sheetfile "sensors.kicad_sch")
-		(attr smd dnp)
+		(attr smd)
 		(fp_line
 			(start -0.153641 0.38)
@@
 		(sheetname "/Schematic/Sensors/")
 		(sheetfile "sensors.kicad_sch")
-		(attr smd dnp)
+		(attr smd)
 		(fp_line
 			(start 3.11 1.11)
@@
 		(sheetname "/Schematic/Sensors/")
 		(sheetfile "sensors.kicad_sch")
-		(attr smd dnp)
+		(attr smd)
 		(fp_line
 			(start 3.11 1.11)
@@
 			)
 		)
-		(property "Value" "DNP-10k"
+		(property "Value" "10k"
 			(at 0 -1.17 90)
 			(layer "B.Fab")
@@
 		(sheetname "/Schematic/Sensors/")
 		(sheetfile "sensors.kicad_sch")
-		(attr smd dnp)
+		(attr smd)
 		(fp_line
 			(start -0.153641 -0.38)
@@
 			)
 		)
-		(property "Value" "DNP-10k"
+		(property "Value" "10k"
 			(at 0 -1.17 90)
 			(layer "B.Fab")
@@
 		(sheetname "/Schematic/Sensors/")
 		(sheetfile "sensors.kicad_sch")
-		(attr smd dnp)
+		(attr smd)
 		(fp_line
 			(start -0.153641 -0.38)
@@
 			)
 		)
-		(property "Value" "DNP-10k"
+		(property "Value" "10k"
 			(at 0 -1.17 90)
 			(layer "B.Fab")
@@
 		(sheetname "/Schematic/Sensors/")
 		(sheetfile "sensors.kicad_sch")
-		(attr smd dnp)
+		(attr smd)
 		(fp_line
 			(start -0.153641 -0.38)
@@
 			)
 		)
-		(property "Value" "DNP-10k"
+		(property "Value" "10k"
 			(at 0 -1.17 90)
 			(layer "B.Fab")
@@
 		(sheetname "/Schematic/Sensors/")
 		(sheetfile "sensors.kicad_sch")
-		(attr smd dnp)
+		(attr smd)
 		(fp_line
 			(start -0.153641 -0.38)
@@
 			)
 		)
-		(property "Value" "DNP-0R"
+		(property "Value" "0R"
 			(at 0 -1.17 0)
 			(layer "B.Fab")
@@
 		(sheetname "/Schematic/Sensors/")
 		(sheetfile "sensors.kicad_sch")
-		(attr smd dnp)
+		(attr smd)
 		(fp_line
 			(start -0.153641 0.38)
@@
 			)
 		)
-		(property "Value" "DNP-10k"
+		(property "Value" "10k"
 			(at 0 -1.17 90)
 			(layer "B.Fab")
@@
 		(sheetname "/Schematic/Sensors/")
 		(sheetfile "sensors.kicad_sch")
-		(attr smd dnp)
+		(attr smd)
 		(fp_line
 			(start -0.153641 -0.38)
@@
 			)
 		)
-		(property "Value" "DNP-10k"
+		(property "Value" "10k"
 			(at 0 -1.17 90)
 			(layer "B.Fab")
@@
 		(sheetname "/Schematic/Sensors/")
 		(sheetfile "sensors.kicad_sch")
-		(attr smd dnp)
+		(attr smd)
 		(fp_line
 			(start -0.153641 -0.38)

Commit message: [verified] feat(hardware): remove upstream brand logos
Parts:
- removed H2: Logo HF 2025, Library_Pollen:Logo_HF_2025
- removed H3: DNP Logo Pollen 2021, Library_Pollen:Logo_Pollen_2021_sq

Commit message: [verified] fix(hardware): correct power bias and default-off GPIO controls
Qualify Q2 land and gate rating, battery-bias LM5050 VS, and correct C39 identity. Add host-referenced active-low battery sensing and default-off amplifier control while preserving connector parity. Expand exact regression guards and complete BOM/position exports. Fabrication approval remains pending physical and runtime validation.
Parts:
- removed D2: 3V3 Zener Diode, Diode_SMD:D_SOD-123
- added Q3: BC847B, Package_TO_SOT_SMD:SOT-23, F.Cu at (111.5, 94.0)
- added Q4: BC847B, Package_TO_SOT_SMD:SOT-23, F.Cu at (115.5, 94.0)
- added Q5: BC847B, Package_TO_SOT_SMD:SOT-23, F.Cu at (118.0, 90.0)
- added R42: 100k, Resistor_SMD:R_0402_1005Metric, F.Cu at (104.0, 93.0)
- added R43: 10k, Resistor_SMD:R_0402_1005Metric, F.Cu at (102.5, 93.0)
- added R44: 10k, Resistor_SMD:R_0402_1005Metric, F.Cu at (108.5, 91.0)
- added R45: 10k, Resistor_SMD:R_0402_1005Metric, F.Cu at (114.5, 90.5)
- added R46: 100k, Resistor_SMD:R_0402_1005Metric, F.Cu at (116.5, 97.5)
- C39: value 100n 6V3 -> 100nF 50V X7R
- Q2: value SI2312CDS-T1-GE3 -> DMN3023L-7; footprint Package_TO_SOT_SMD:TSOT-23 -> Package_TO_SOT_SMD:DMN3023L_SOT23_Diodes
- R24: value 10k -> 100k
- R3: value 0R -> 10k
Connections:
- net Net-(U1-~{SHND}) renamed AMP_SHDN
- J4 pad 11: unconnected-(J4-Pin_11-Pad11) -> AMP_ENABLE
- R24 pad 1: /Schematic/Audio/GPIO3_B4_P31 -> BAT_BASE
- R8 pad 1: +5V -> +BATT
Routing:
- net AMP_BASE: track 0.00 -> 33.8 mm, vias 0 -> 3
- net AMP_ENABLE: track 0.00 -> 26.7 mm, vias 0 -> 2
- net AMP_INHIBIT: track 0.00 -> 26.3 mm, vias 0 -> 4
- net BAT_BASE: track 0.00 -> 15.0 mm, vias 0 -> 2
- net /Schematic/Audio/GPIO3_B4_P31: track 29.3 -> 38.9 mm, vias 3 -> 5
- net GND: track 109.3 -> 118.6 mm, vias 40 -> 43
- net +BATT: track 38.9 -> 48.0 mm, vias 1 -> 2
- net AMP_SHDN: track 1.75 -> 6.72 mm, vias 0 -> 1
- net +5V: track 133.5 -> 135.7 mm, vias 6 -> 7
- net +3V3: track 210.1 -> 211.1 mm
